File: Hardware/DCC-light.brd (EAGLE design)
At the start: 13 x 11.5 mm, 22 parts, among them Q1 MOSFET-NCHANNEL2N7002PW, U1 G2X[2/3]1---RSA16, U2 SPX3819M5-L-3-3, U3 24LC00OT, U4 BGX50A

Commit message: Update hardware design
Parts:
- R1: value 4.7K -> 47K
- R6, R8: value 4.7K -> 9.1K
- R7, R9: value 4.7K -> 2.7K
Changed lines of the file:
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@@
 <attribute name="VALUE" x="10.3124" y="10.3378" size="0.4064" layer="28" font="vector" rot="MR180"/>
 </element>
-<element name="R1" library="adafruit" package="R0402" value="4.7K" x="11.303" y="8.509" smashed="yes">
+<element name="R1" library="adafruit" package="R0402" value="47K" x="11.303" y="8.509" smashed="yes">
 <attribute name="NAME" x="11.0744" y="3.175" size="0.8128" layer="25" font="vector"/>
 <attribute name="VALUE" x="10.668" y="6.477" size="1.27" layer="27"/>
@@
 <attribute name="VALUE" x="10.0711" y="8.6106" size="0.4064" layer="28" rot="MR180"/>
 </element>
-<element name="R6" library="adafruit" package="R0402" value="4.7K" x="8.7884" y="2.8448" smashed="yes" rot="MR180">
+<element name="R6" library="adafruit" package="R0402" value="9.1K" x="8.7884" y="2.8448" smashed="yes" rot="MR180">
 <attribute name="NAME" x="8.7884" y="0.9398" size="0.8128" layer="26" font="vector" rot="MR180"/>
 <attribute name="VALUE" x="8.1534" y="4.8768" size="1.27" layer="28" rot="MR180"/>
 </element>
-<element name="R7" library="adafruit" package="R0402" value="4.7K" x="8.7884" y="3.9624" smashed="yes" rot="MR0">
+<element name="R7" library="adafruit" package="R0402" value="2.7K" x="8.7884" y="3.9624" smashed="yes" rot="MR0">
 <attribute name="NAME" x="10.2616" y="1.1938" size="0.8128" layer="26" font="vector" rot="MR0"/>
 <attribute name="VALUE" x="9.4234" y="1.9304" size="1.27" layer="28" rot="MR0"/>
 </element>
-<element name="R8" library="adafruit" package="R0402" value="4.7K" x="1.9812" y="4.953" smashed="yes" rot="MR0">
+<element name="R8" library="adafruit" package="R0402" value="9.1K" x="1.9812" y="4.953" smashed="yes" rot="MR0">
 <attribute name="NAME" x="4.4196" y="5.9944" size="0.8128" layer="26" font="vector" rot="MR0"/>
 <attribute name="VALUE" x="2.6162" y="2.921" size="1.27" layer="28" rot="MR0"/>
 </element>
-<element name="R9" library="adafruit" package="R0402" value="4.7K" x="1.9304" y="6.1976" smashed="yes" rot="MR180">
+<element name="R9" library="adafruit" package="R0402" value="2.7K" x="1.9304" y="6.1976" smashed="yes" rot="MR180">
 <attribute name="NAME" x="3.0226" y="5.8674" size="0.8128" layer="26" font="vector" rot="MR180"/>
 <attribute name="VALUE" x="1.2954" y="8.2296" size="1.27" layer="28" rot="MR180"/>
@@
 <contactref element="R4" pad="1"/>
 <polygon width="0.2032" layer="16">
-<vertex x="-1.143" y="15.24"/>
-<vertex x="25.4" y="15.24"/>
-<vertex x="25.654" y="4.572"/>
-<vertex x="-1.143" y="4.572"/>
+<vertex x="0.127" y="11.43"/>
+<vertex x="12.954" y="11.43"/>
+<vertex x="12.954" y="4.572"/>
+<vertex x="0.127" y="4.572"/>
 </polygon>
 <polygon width="0.2032" layer="1">
-<vertex x="-1.143" y="15.24"/>
-<vertex x="25.4" y="15.24"/>
-<vertex x="25.4" y="-1.397"/>
-<vertex x="-1.27" y="-1.397"/>
-<vertex x="-1.27" y="2.54"/>
+<vertex x="0.127" y="11.43"/>
+<vertex x="12.954" y="11.43"/>
+<vertex x="12.954" y="0.127"/>
+<vertex x="0" y="0.127"/>
 </polygon>
 <contactref element="JP1" pad="4"/>
@@
 <via x="5.1562" y="1.905" extent="1-16" drill="0.3"/>
 <polygon width="0.254" layer="16">
-<vertex x="4.064" y="-0.508"/>
-<vertex x="8.636" y="-0.508"/>
+<vertex x="4.064" y="0.254"/>
+<vertex x="8.636" y="0.254"/>
 <vertex x="8.636" y="3.81"/>
 <vertex x="4.064" y="3.81"/>
