File: Hardware/DCC-command-center-V2.brd (EAGLE design)
At the start: 100 x 53.6 mm, 211 parts, among them U1 LM339, U2 LM339, U3 LM339, U4 LM339, U5 LM339, U6 LM339, U7 DRV8801

Commit message: Update component values
Parts:
- R1, R10, R11, R12, R17, R18, R19, R2, R20, R25, R26, R27, R28, R3, R33, R34, R35, R36, R4, R41, R42, R43, R44, R9: value 68R -> DNP
- VR1, VR10, VR11, VR12, VR13, VR14, VR15, VR16, VR17, VR18, VR19, VR2, VR20, VR21, VR22, VR23, VR24, VR3, VR4, VR5, VR6, VR7, VR8, VR9: value 100K -> 10K
